Commit message: buggy code just to test if arm can move

File: mvp_arm_6dof_description/urdf/mvp_arm_6dof.xacro (robot description, xacro)
@@ -1,19 +1,13 @@
 <?xml version="1.0" ?>
 <robot name="mvp_arm_6dof" xmlns:xacro="http://www.ros.org/wiki/xacro">
-	<!--
-	     ADDED DUMMY LINK AND DUMMMY JOINT
-	     -->
 <xacro:include filename="$(find mvp_arm_6dof_description)/urdf/materials.xacro" />
 <xacro:include filename="$(find mvp_arm_6dof_description)/urdf/mvp_arm_6dof.trans" />
 <xacro:include filename="$(find mvp_arm_6dof_description)/urdf/mvp_arm_6dof.gazebo" />
-<!-- dummy link below -->
-<link name="dummy">
-</link>
-<!-- dummy link above -->
+<link name="world"/>
 <link name="base_link">
   <inertial>
-    <origin rpy="0 0 0" xyz="1.5273427923512274e-08 -0.0012615194115251204 0.015200351763726439"/>
-    <mass value="1.6606259711147333"/>
-    <inertia ixx="0.006748" ixy="0.0" ixz="-0.0" iyy="0.007016" iyz="4.2e-05" izz="0.012699"/>
+		<origin xyz="0 0 0" rpy="0 0 0" />
+		<mass value="3.06" />
+		<inertia ixx="0.3" ixy="0.0" ixz="0.0" iyy="0.3" iyz="0.0" izz="0.3" />
   </inertial>
   <visual>
@@ -33,7 +27,7 @@
 <link name="f3Bracket_1">
   <inertial>
-    <origin rpy="0 0 0" xyz="0.0018413874270871398 8.06819888676813e-15 2.0816681711721685e-17"/>
-    <mass value="0.0016262220015435807"/>
-    <inertia ixx="0.0" ixy="-0.0" ixz="-0.0" iyy="0.0" iyz="0.0" izz="0.0"/>
+		<origin xyz="0 0 0" rpy="0 0 0" />
+		<mass value="3.06" />
+		<inertia ixx="0.3" ixy="0.0" ixz="0.0" iyy="0.3" iyz="0.0" izz="0.3" />
   </inertial>
   <visual>
@@ -53,7 +47,7 @@
 <link name="f3Bracket__1__1">
   <inertial>
-    <origin rpy="0 0 0" xyz="-0.0018413874270886074 6.831341048396666e-15 -3.469446951953614e-17"/>
-    <mass value="0.0016262220015435807"/>
-    <inertia ixx="0.0" ixy="0.0" ixz="0.0" iyy="0.0" iyz="-0.0" izz="0.0"/>
+		<origin xyz="0 0 0" rpy="0 0 0" />
+		<mass value="3.06" />
+		<inertia ixx="0.3" ixy="0.0" ixz="0.0" iyy="0.3" iyz="0.0" izz="0.3" />
   </inertial>
   <visual>
@@ -73,7 +67,7 @@
 <link name="AX12A_servo_1">
   <inertial>
-    <origin rpy="0 0 0" xyz="0.01350070935914761 -0.005876867522658821 -0.01479497142329602"/>
-    <mass value="0.3366787209762054"/>
-    <inertia ixx="9.7e-05" ixy="-0.0" ixz="-0.0" iyy="5.4e-05" iyz="-1e-06" izz="8.2e-05"/>
+		<origin xyz="0 0 0" rpy="0 0 0" />
+		<mass value="3.06" />
+		<inertia ixx="0.3" ixy="0.0" ixz="0.0" iyy="0.3" iyz="0.0" izz="0.3" />
   </inertial>
   <visual>
@@ -93,7 +87,7 @@
 <link name="lid_1">
   <inertial>
-    <origin rpy="0 0 0" xyz="-1.0658141036401502e-15 2.4713564528155986e-15 0.0024995000000005013"/>
-    <mass value="0.7384184020105663"/>
-    <inertia ixx="0.001114" ixy="0.0" ixz="0.0" iyy="0.001114" iyz="-0.0" izz="0.002224"/>
+		<origin xyz="0 0 0" rpy="0 0 0" />
+		<mass value="3.06" />
+		<inertia ixx="0.3" ixy="0.0" ixz="0.0" iyy="0.3" iyz="0.0" izz="0.3" />
   </inertial>
   <visual>
@@ -113,7 +107,7 @@
 <link name="f3Bracket__2__1">
   <inertial>
-    <origin rpy="0 0 0" xyz="-4.2188474935755947e-16 8.477663016037695e-15 0.0018408874270881004"/>
-    <mass value="0.0016262220015435807"/>
-    <inertia ixx="0.0" ixy="0.0" ixz="0.0" iyy="0.0" iyz="-0.0" izz="0.0"/>
+		<origin xyz="0 0 0" rpy="0 0 0" />
+		<mass value="3.06" />
+		<inertia ixx="0.3" ixy="0.0" ixz="0.0" iyy="0.3" iyz="0.0" izz="0.3" />
   </inertial>
   <visual>
@@ -133,7 +127,7 @@
 <link name="AX12A_servo__1__1">
   <inertial>
-    <origin rpy="0 0 0" xyz="0.014794971423295564 0.007999290640854232 0.02337263247733931"/>
-    <mass value="0.3366787209762054"/>
-    <inertia ixx="8.2e-05" ixy="-0.0" ixz="1e-06" iyy="9.7e-05" iyz="0.0" izz="5.4e-05"/>
+		<origin xyz="0 0 0" rpy="0 0 0" />
+		<mass value="3.06" />
+		<inertia ixx="0.3" ixy="0.0" ixz="0.0" iyy="0.3" iyz="0.0" izz="0.3" />
   </inertial>
   <visual>
@@ -153,7 +147,7 @@
 <link name="f2Bracket_1">
   <inertial>
-    <origin rpy="0 0 0" xyz="0.02099999999999843 0.011463049476928342 0.011458018229762487"/>
-    <mass value="0.0037556666472927302"/>
-    <inertia ixx="1e-06" ixy="0.0" ixz="-0.0" iyy="2e-06" iyz="-0.0" izz="2e-06"/>
+		<origin xyz="0 0 0" rpy="0 0 0" />
+		<mass value="3.06" />
+		<inertia ixx="0.3" ixy="0.0" ixz="0.0" iyy="0.3" iyz="0.0" izz="0.3" />
   </inertial>
   <visual>
@@ -173,7 +167,7 @@
 <link name="shoulderArm__1">
   <inertial>
-    <origin rpy="0 0 0" xyz="1.7088652541630278e-15 0.05303289486060747 0.05303290188896653"/>
-    <mass value="1.4306625"/>
-    <inertia ixx="0.002769" ixy="-0.0" ixz="-0.0" iyy="0.001626" iyz="-0.001298" izz="0.001626"/>
+		<origin xyz="0 0 0" rpy="0 0 0" />
+		<mass value="3.06" />
+		<inertia ixx="0.3" ixy="0.0" ixz="0.0" iyy="0.3" iyz="0.0" izz="0.3" />
   </inertial>
   <visual>
@@ -193,7 +187,7 @@
 <link name="f3Bracket__3__1">
   <inertial>
-    <origin rpy="0 0 0" xyz="5.250465860695552e-15 0.0013019609860796533 0.0013019680144470969"/>
-    <mass value="0.0016262220015435807"/>
-    <inertia ixx="0.0" ixy="-0.0" ixz="0.0" iyy="0.0" iyz="0.0" izz="0.0"/>
+		<origin xyz="0 0 0" rpy="0 0 0" />
+		<mass value="3.06" />
+		<inertia ixx="0.3" ixy="0.0" ixz="0.0" iyy="0.3" iyz="0.0" izz="0.3" />
   </inertial>
   <visual>
@@ -213,7 +207,7 @@
 <link name="AX12A_servo__2__1">
   <inertial>
-    <origin rpy="0 0 0" xyz="0.01479397142330254 0.010869789625758658 0.02218479983944499"/>
-    <mass value="0.3366787209762054"/>
-    <inertia ixx="8.2e-05" ixy="1e-06" ixz="1e-06" iyy="7.6e-05" iyz="-2.2e-05" izz="7.6e-05"/>
+		<origin xyz="0 0 0" rpy="0 0 0" />
+		<mass value="3.06" />
+		<inertia ixx="0.3" ixy="0.0" ixz="0.0" iyy="0.3" iyz="0.0" izz="0.3" />
   </inertial>
   <visual>
@@ -233,7 +227,7 @@
 <link name="f2Bracket__1__1">
   <inertial>
-    <origin rpy="0 0 0" xyz="0.02099900000000768 -0.011458683360921401 0.011462891374124484"/>
-    <mass value="0.0037556666472927302"/>
-    <inertia ixx="1e-06" ixy="0.0" ixz="0.0" iyy="2e-06" iyz="0.0" izz="2e-06"/>
+		<origin xyz="0 0 0" rpy="0 0 0" />
+		<mass value="3.06" />
+		<inertia ixx="0.3" ixy="0.0" ixz="0.0" iyy="0.3" iyz="0.0" izz="0.3" />
   </inertial>
   <visual>
@@ -253,7 +247,7 @@
 <link name="axis3-4_connector__1">
   <inertial>
-    <origin rpy="0 0 0" xyz="7.741767021180422e-09 -0.013131073230303991 0.013131242967982293"/>
-    <mass value="0.2107220147290529"/>
-    <inertia ixx="0.000131" ixy="-0.0" ixz="0.0" iyy="9.2e-05" iyz="-1.3e-05" izz="9.2e-05"/>
+		<origin xyz="0 0 0" rpy="0 0 0" />
+		<mass value="3.06" />
+		<inertia ixx="0.3" ixy="0.0" ixz="0.0" iyy="0.3" iyz="0.0" izz="0.3" />
   </inertial>
   <visual>
@@ -273,7 +267,7 @@
 <link name="f3Bracket__4__1">
   <inertial>
-    <origin rpy="0 0 0" xyz="8.331551594464859e-15 0.006959286311871121 -0.00435505918631085"/>
-    <mass value="0.0016262220015435807"/>
-    <inertia ixx="0.0" ixy="0.0" ixz="-0.0" iyy="0.0" iyz="0.0" izz="0.0"/>
+		<origin xyz="0 0 0" rpy="0 0 0" />
+		<mass value="3.06" />
+		<inertia ixx="0.3" ixy="0.0" ixz="0.0" iyy="0.3" iyz="0.0" izz="0.3" />
   </inertial>
   <visual>
@@ -293,7 +287,7 @@
 <link name="f3Bracket__5__1">
   <inertial>
-    <origin rpy="0 0 0" xyz="1.960920575222458e-14 0.004355228923988971 -0.006959116574192292"/>
-    <mass value="0.0016262220015435807"/>
-    <inertia ixx="0.0" ixy="0.0" ixz="-0.0" iyy="0.0" iyz="0.0" izz="0.0"/>
+		<origin xyz="0 0 0" rpy="0 0 0" />
+		<mass value="3.06" />
+		<inertia ixx="0.3" ixy="0.0" ixz="0.0" iyy="0.3" iyz="0.0" izz="0.3" />
   </inertial>
   <visual>
@@ -313,7 +307,7 @@
 <link name="AX12A_servo__3__1">
   <inertial>
-    <origin rpy="0 0 0" xyz="-0.005876867522646675 0.0009146721471553626 -0.020007505594804464"/>
-    <mass value="0.3366787209762054"/>
-    <inertia ixx="5.4e-05" ixy="1e-06" ixz="-1e-06" iyy="9e-05" iyz="8e-06" izz="9e-05"/>
+		<origin xyz="0 0 0" rpy="0 0 0" />
+		<mass value="3.06" />
+		<inertia ixx="0.3" ixy="0.0" ixz="0.0" iyy="0.3" iyz="0.0" izz="0.3" />
   </inertial>
   <visual>
@@ -333,7 +327,7 @@
 <link name="f3Bracket__6__1">
   <inertial>
-    <origin rpy="0 0 0" xyz="1.7957857423311907e-14 -0.001301912074779893 0.0013020818124673261"/>
-    <mass value="0.0016262220015435807"/>
-    <inertia ixx="0.0" ixy="-0.0" ixz="0.0" iyy="0.0" iyz="-0.0" izz="0.0"/>
+		<origin xyz="0 0 0" rpy="0 0 0" />
+		<mass value="3.06" />
+		<inertia ixx="0.3" ixy="0.0" ixz="0.0" iyy="0.3" iyz="0.0" izz="0.3" />
   </inertial>
   <visual>
@@ -353,7 +347,7 @@
 <link name="axis4ARM__1">
   <inertial>
-    <origin rpy="0 0 0" xyz="2.929601006229632e-14 -0.053032748695814015 0.05303291843349328"/>
-    <mass value="0.9125625000000004"/>
-    <inertia ixx="0.001759" ixy="0.0" ixz="-0.0" iyy="0.000952" iyz="0.000832" izz="0.000952"/>
+		<origin xyz="0 0 0" rpy="0 0 0" />
+		<mass value="3.06" />
+		<inertia ixx="0.3" ixy="0.0" ixz="0.0" iyy="0.3" iyz="0.0" izz="0.3" />
   </inertial>
   <visual>
@@ -373,7 +367,7 @@
 <link name="f3Bracket__7__1">
   <inertial>
-    <origin rpy="0 0 0" xyz="4.110253803979447e-14 -0.0013018148212854495 0.001301984558973679"/>
-    <mass value="0.0016262220015435807"/>
-    <inertia ixx="0.0" ixy="-0.0" ixz="0.0" iyy="0.0" iyz="-0.0" izz="0.0"/>
+		<origin xyz="0 0 0" rpy="0 0 0" />
+		<mass value="3.06" />
+		<inertia ixx="0.3" ixy="0.0" ixz="0.0" iyy="0.3" iyz="0.0" izz="0.3" />
   </inertial>
   <visual>
@@ -393,7 +387,7 @@
 <link name="AX12A_servo__4__1">
   <inertial>
-    <origin rpy="0 0 0" xyz="0.014793971423341353 -0.010870646646293183 0.022183813198644264"/>
-    <mass value="0.3366787209762054"/>
-    <inertia ixx="8.2e-05" ixy="-1e-06" ixz="1e-06" iyy="7.6e-05" iyz="2.2e-05" izz="7.6e-05"/>
+		<origin xyz="0 0 0" rpy="0 0 0" />
+		<mass value="3.06" />
+		<inertia ixx="0.3" ixy="0.0" ixz="0.0" iyy="0.3" iyz="0.0" izz="0.3" />
   </inertial>
   <visual>
@@ -413,7 +407,7 @@
 <link name="f2Bracket__2__1">
   <inertial>
-    <origin rpy="0 0 0" xyz="0.020999000000046463 -0.011462738180973452 -0.011458659788035952"/>
-    <mass value="0.0037556666472927302"/>
-    <inertia ixx="1e-06" ixy="-0.0" ixz="0.0" iyy="2e-06" iyz="-0.0" izz="2e-06"/>
+		<origin xyz="0 0 0" rpy="0 0 0" />
+		<mass value="3.06" />
+		<inertia ixx="0.3" ixy="0.0" ixz="0.0" iyy="0.3" iyz="0.0" izz="0.3" />
   </inertial>
   <visual>
@@ -433,7 +427,7 @@
 <link name="axis5-6_connector__1">
   <inertial>
-    <origin rpy="0 0 0" xyz="-2.2518098496959738e-13 -0.013131095249087704 -0.01313104418317057"/>
-    <mass value="0.2107220147290529"/>
-    <inertia ixx="8e-05" ixy="-0.0" ixz="0.0" iyy="0.000118" iyz="-1.3e-05" izz="0.000118"/>
+		<origin xyz="0 0 0" rpy="0 0 0" />
+		<mass value="3.06" />
+		<inertia ixx="0.3" ixy="0.0" ixz="0.0" iyy="0.3" iyz="0.0" izz="0.3" />
   </inertial>
   <visual>
@@ -453,7 +447,7 @@
 <link name="f3Bracket__9__1">
   <inertial>
-    <origin rpy="0 0 0" xyz="0.001841387427043583 0.005657241073397323 0.005657281190819818"/>
-    <mass value="0.0016262220015435807"/>
-    <inertia ixx="0.0" ixy="-0.0" ixz="-0.0" iyy="0.0" iyz="-0.0" izz="0.0"/>
+		<origin xyz="0 0 0" rpy="0 0 0" />
+		<mass value="3.06" />
+		<inertia ixx="0.3" ixy="0.0" ixz="0.0" iyy="0.3" iyz="0.0" izz="0.3" />
   </inertial>
   <visual>
@@ -473,7 +467,7 @@
 <link name="f3Bracket__8__1">
   <inertial>
-    <origin rpy="0 0 0" xyz="-0.0018413874273180211 0.0056572410733904815 0.005657281190812213"/>
-    <mass value="0.0016262220015435807"/>
-    <inertia ixx="0.0" ixy="-0.0" ixz="-0.0" iyy="0.0" iyz="-0.0" izz="0.0"/>
+		<origin xyz="0 0 0" rpy="0 0 0" />
+		<mass value="3.06" />
+		<inertia ixx="0.3" ixy="0.0" ixz="0.0" iyy="0.3" iyz="0.0" izz="0.3" />
   </inertial>
   <visual>
@@ -493,7 +487,7 @@
 <link name="AX12A_servo__5__1">
   <inertial>
-    <origin rpy="0 0 0" xyz="-0.013499290641083328 0.014616875823199357 0.006305478684788701"/>
-    <mass value="0.3366787209762054"/>
-    <inertia ixx="9.7e-05" ixy="0.0" ixz="0.0" iyy="6.6e-05" iyz="1.4e-05" izz="6.9e-05"/>
+		<origin xyz="0 0 0" rpy="0 0 0" />
+		<mass value="3.06" />
+		<inertia ixx="0.3" ixy="0.0" ixz="0.0" iyy="0.3" iyz="0.0" izz="0.3" />
   </inertial>
   <visual>
@@ -513,7 +507,7 @@
 <link name="f3Bracket__10__1">
   <inertial>
-    <origin rpy="0 0 0" xyz="-2.483881156312151e-13 -0.001301753641823486 -0.0013020634793980412"/>
-    <mass value="0.0016262220015435807"/>
-    <inertia ixx="0.0" ixy="-0.0" ixz="0.0" iyy="0.0" iyz="0.0" izz="0.0"/>
+		<origin xyz="0 0 0" rpy="0 0 0" />
+		<mass value="3.06" />
+		<inertia ixx="0.3" ixy="0.0" ixz="0.0" iyy="0.3" iyz="0.0" izz="0.3" />
   </inertial>
   <visual>
@@ -533,7 +527,7 @@
 <link name="AX12A_servo__6__1">
   <inertial>
-    <origin rpy="0 0 0" xyz="0.007999290640599755 -0.02865305003000715 -0.004402427555891486"/>
-    <mass value="0.3366787209762054"/>
-    <inertia ixx="9.7e-05" ixy="-0.0" ixz="0.0" iyy="6.6e-05" iyz="-1.4e-05" izz="6.9e-05"/>
+		<origin xyz="0 0 0" rpy="0 0 0" />
+		<mass value="3.06" />
+		<inertia ixx="0.3" ixy="0.0" ixz="0.0" iyy="0.3" iyz="0.0" izz="0.3" />
   </inertial>
   <visual>
@@ -552,6 +546,6 @@
 </link>
 <!-- dummy joint below -->
-<joint name="dummy_joint" type="fixed">
-  <parent link="dummy"/>
+<joint name="world" type="fixed">
+  <parent link="world"/>
   <child link="base_link"/>
  </joint>
@@ -577,4 +571,5 @@
   <child link="lid_1"/>
   <axis xyz="0.0 0.0 -1.0"/>
+	<dynamics damping="1.0"/>
 </joint>
 <joint name="Rigid18" type="fixed">
@@ -593,4 +588,5 @@
   <child link="f2Bracket_1"/>
   <axis xyz="1.0 -0.0 0.0"/>
+	<dynamics damping="1.0"/>
 </joint>
 <joint name="Rigid23" type="fixed">
@@ -614,4 +610,5 @@
   <child link="f2Bracket__1__1"/>
   <axis xyz="1.0 0.0 -0.0"/>
+	<dynamics damping="1.0"/>
 </joint>
 <joint name="Rigid32" type="fixed">
@@ -640,4 +637,5 @@
   <child link="f3Bracket__6__1"/>
   <axis xyz="-0.0 0.707107 -0.707107"/>
+	<dynamics damping="1.0"/>
 </joint>
 <joint name="Rigid37" type="fixed">
@@ -661,4 +659,5 @@
   <child link="f2Bracket__2__1"/>
   <axis xyz="1.0 0.0 -0.0"/>
+	<dynamics damping="1.0"/>
 </joint>
 <joint name="Rigid41" type="fixed">
@@ -687,4 +686,5 @@
   <child link="f3Bracket__10__1"/>
   <axis xyz="-0.0 -0.707107 -0.707107"/>
+	<dynamics damping="1.0"/>
 </joint>
 <joint name="Rigid46" type="fixed">
