Commit message: updated 6dof v2 description

File: mvp_arm_6dof_v4_description/urdf/materials.xacro (robot description, xacro)
@@ -1,5 +1,5 @@
 <?xml version="1.0" ?>
 <robot name="mvp_arm_6dof_v4" xmlns:xacro="http://www.ros.org/wiki/xacro" >
-<material name="silver_default">
+<material name="silver">
   <color rgba="0.700 0.700 0.700 1.000"/>
 </material>

File: mvp_arm_6dof_v4_description/urdf/mvp_arm_6dof_v4.xacro (robot description, xacro)
@@ -15,5 +15,5 @@
       <mesh filename="package://mvp_arm_6dof_v4_description/meshes/base_link.stl" scale="0.001 0.001 0.001"/>
     </geometry>
-    <material name="silver_default"/>
+    <material name="silver"/>
   </visual>
   <collision>
@@ -24,3 +24,685 @@
   </collision>
 </link>
+<link name="f3Bracket_1">
+  <inertial>
+    <origin rpy="0 0 0" xyz="0.0018413874270871398 8.06819888676813e-15 2.0816681711721685e-17"/>
+    <mass value="0.0016262220015435807"/>
+    <inertia ixx="0.0" ixy="-0.0" ixz="-0.0" iyy="0.0" iyz="0.0" izz="0.0"/>
+  </inertial>
+  <visual>
+    <origin rpy="0 0 0" xyz="0.019 0.01475 -0.041"/>
+    <geometry>
+      <mesh filename="package://mvp_arm_6dof_v4_description/meshes/f3Bracket_1.stl" scale="0.001 0.001 0.001"/>
+    </geometry>
+    <material name="silver"/>
+  </visual>
+  <collision>
+    <origin rpy="0 0 0" xyz="0.019 0.01475 -0.041"/>
+    <geometry>
+      <mesh filename="package://mvp_arm_6dof_v4_description/meshes/f3Bracket_1.stl" scale="0.001 0.001 0.001"/>
+    </geometry>
+  </collision>
+</link>
+<link name="f3Bracket__1__1">
+  <inertial>
+    <origin rpy="0 0 0" xyz="-0.0018413874270886074 6.831341048396666e-15 -3.469446951953614e-17"/>
+    <mass value="0.0016262220015435807"/>
+    <inertia ixx="0.0" ixy="0.0" ixz="0.0" iyy="0.0" iyz="-0.0" izz="0.0"/>
+  </inertial>
+  <visual>
+    <origin rpy="0 0 0" xyz="-0.019 0.01475 -0.041"/>
+    <geometry>
+      <mesh filename="package://mvp_arm_6dof_v4_description/meshes/f3Bracket__1__1.stl" scale="0.001 0.001 0.001"/>
+    </geometry>
+    <material name="silver"/>
+  </visual>
+  <collision>
+    <origin rpy="0 0 0" xyz="-0.019 0.01475 -0.041"/>
+    <geometry>
+      <mesh filename="package://mvp_arm_6dof_v4_description/meshes/f3Bracket__1__1.stl" scale="0.001 0.001 0.001"/>
+    </geometry>
+  </collision>
+</link>
+<link name="AX12A_servo_1">
+  <inertial>
+    <origin rpy="0 0 0" xyz="0.013500709359147614 -0.005876867522658821 -0.01479497142329602"/>
+    <mass value="0.3366787209762054"/>
+    <inertia ixx="9.7e-05" ixy="-0.0" ixz="-0.0" iyy="5.4e-05" iyz="-1e-06" izz="8.2e-05"/>
+  </inertial>
+  <visual>
+    <origin rpy="0 0 0" xyz="0.0135 0.00675 -0.057"/>
+    <geometry>
+      <mesh filename="package://mvp_arm_6dof_v4_description/meshes/AX12A_servo_1.stl" scale="0.001 0.001 0.001"/>
+    </geometry>
+    <material name="silver"/>
+  </visual>
+  <collision>
+    <origin rpy="0 0 0" xyz="0.0135 0.00675 -0.057"/>
+    <geometry>
+      <mesh filename="package://mvp_arm_6dof_v4_description/meshes/AX12A_servo_1.stl" scale="0.001 0.001 0.001"/>
+    </geometry>
+  </collision>
+</link>
+<link name="base_lid__1">
+  <inertial>
+    <origin rpy="0 0 0" xyz="-3.907985046680551e-16 1.8474111129762605e-15 0.0024995000000005013"/>
+    <mass value="0.7384184020105663"/>
+    <inertia ixx="0.001114" ixy="-0.0" ixz="0.0" iyy="0.001114" iyz="0.0" izz="0.002224"/>
+  </inertial>
+  <visual>
+    <origin rpy="0 0 0" xyz="0.0 -0.0 -0.06175"/>
+    <geometry>
+      <mesh filename="package://mvp_arm_6dof_v4_description/meshes/base_lid__1.stl" scale="0.001 0.001 0.001"/>
+    </geometry>
+    <material name="silver"/>
+  </visual>
+  <collision>
+    <origin rpy="0 0 0" xyz="0.0 -0.0 -0.06175"/>
+    <geometry>
+      <mesh filename="package://mvp_arm_6dof_v4_description/meshes/base_lid__1.stl" scale="0.001 0.001 0.001"/>
+    </geometry>
+  </collision>
+</link>
+<link name="f3Bracket__2__1">
+  <inertial>
+    <origin rpy="0 0 0" xyz="-6.31050767196939e-15 2.4780177909633494e-15 0.0018408874270881143"/>
+    <mass value="0.0016262220015435807"/>
+    <inertia ixx="0.0" ixy="-0.0" ixz="0.0" iyy="0.0" iyz="0.0" izz="0.0"/>
+  </inertial>
+  <visual>
+    <origin rpy="0 0 0" xyz="0.0 -0.0 -0.06675"/>
+    <geometry>
+      <mesh filename="package://mvp_arm_6dof_v4_description/meshes/f3Bracket__2__1.stl" scale="0.001 0.001 0.001"/>
+    </geometry>
+    <material name="silver"/>
+  </visual>
+  <collision>
+    <origin rpy="0 0 0" xyz="0.0 -0.0 -0.06675"/>
+    <geometry>
+      <mesh filename="package://mvp_arm_6dof_v4_description/meshes/f3Bracket__2__1.stl" scale="0.001 0.001 0.001"/>
+    </geometry>
+  </collision>
+</link>
+<link name="AX12A_servo__1__1">
+  <inertial>
+    <origin rpy="0 0 0" xyz="-0.007999290640852062 0.01479397142329844 0.02337263247733931"/>
+    <mass value="0.3366787209762054"/>
+    <inertia ixx="9.7e-05" ixy="0.0" ixz="-0.0" iyy="8.2e-05" iyz="1e-06" izz="5.4e-05"/>
+  </inertial>
+  <visual>
+    <origin rpy="0 0 0" xyz="-0.008 0.015999 -0.07225"/>
+    <geometry>
+      <mesh filename="package://mvp_arm_6dof_v4_description/meshes/AX12A_servo__1__1.stl" scale="0.001 0.001 0.001"/>
+    </geometry>
+    <material name="silver"/>
+  </visual>
+  <collision>
+    <origin rpy="0 0 0" xyz="-0.008 0.015999 -0.07225"/>
+    <geometry>
+      <mesh filename="package://mvp_arm_6dof_v4_description/meshes/AX12A_servo__1__1.stl" scale="0.001 0.001 0.001"/>
+    </geometry>
+  </collision>
+</link>
+<link name="f2Bracket_1">
+  <inertial>
+    <origin rpy="0 0 0" xyz="-3.2040755970985657e-06 0.020999000000001256 0.016207495960826337"/>
+    <mass value="0.0037556666472927302"/>
+    <inertia ixx="2e-06" ixy="-0.0" ixz="0.0" iyy="1e-06" iyz="0.0" izz="1e-06"/>
+  </inertial>
+  <visual>
+    <origin rpy="0 0 0" xyz="0.0 0.020749 -0.10825"/>
+    <geometry>
+      <mesh filename="package://mvp_arm_6dof_v4_description/meshes/f2Bracket_1.stl" scale="0.001 0.001 0.001"/>
+    </geometry>
+    <material name="silver"/>
+  </visual>
+  <collision>
+    <origin rpy="0 0 0" xyz="0.0 0.020749 -0.10825"/>
+    <geometry>
+      <mesh filename="package://mvp_arm_6dof_v4_description/meshes/f2Bracket_1.stl" scale="0.001 0.001 0.001"/>
+    </geometry>
+  </collision>
+</link>
+<link name="shoulderArm__1">
+  <inertial>
+    <origin rpy="0 0 0" xyz="4.087757237730653e-07 4.462142461081342e-15 0.07500026947793709"/>
+    <mass value="1.4306625"/>
+    <inertia ixx="0.002924" ixy="0.0" ixz="-0.0" iyy="0.002769" iyz="-0.0" izz="0.000328"/>
+  </inertial>
+  <visual>
+    <origin rpy="0 0 0" xyz="5e-06 -0.00025 -0.134703"/>
+    <geometry>
+      <mesh filename="package://mvp_arm_6dof_v4_description/meshes/shoulderArm__1.stl" scale="0.001 0.001 0.001"/>
+    </geometry>
+    <material name="silver"/>
+  </visual>
+  <collision>
+    <origin rpy="0 0 0" xyz="5e-06 -0.00025 -0.134703"/>
+    <geometry>
+      <mesh filename="package://mvp_arm_6dof_v4_description/meshes/shoulderArm__1.stl" scale="0.001 0.001 0.001"/>
+    </geometry>
+  </collision>
+</link>
+<link name="f3Bracket__3__1">
+  <inertial>
+    <origin rpy="0 0 0" xyz="4.0877572965058626e-07 7.941618283130447e-15 0.0018416569050248022"/>
+    <mass value="0.0016262220015435807"/>
+    <inertia ixx="0.0" ixy="0.0" ixz="-0.0" iyy="0.0" iyz="0.0" izz="0.0"/>
+  </inertial>
+  <visual>
+    <origin rpy="0 0 0" xyz="5e-06 -0.00025 -0.284703"/>
+    <geometry>
+      <mesh filename="package://mvp_arm_6dof_v4_description/meshes/f3Bracket__3__1.stl" scale="0.001 0.001 0.001"/>
+    </geometry>
+    <material name="silver"/>
+  </visual>
+  <collision>
+    <origin rpy="0 0 0" xyz="5e-06 -0.00025 -0.284703"/>
+    <geometry>
+      <mesh filename="package://mvp_arm_6dof_v4_description/meshes/f3Bracket__3__1.stl" scale="0.001 0.001 0.001"/>
+    </geometry>
+  </collision>
+</link>
+<link name="AX12A_servo__2__1">
+  <inertial>
+    <origin rpy="0 0 0" xyz="0.008001118134871487 0.014793971423305203 0.02337340195527582"/>
+    <mass value="0.3366787209762054"/>
+    <inertia ixx="9.7e-05" ixy="0.0" ixz="-0.0" iyy="8.2e-05" iyz="1e-06" izz="5.4e-05"/>
+  </inertial>
+  <visual>
+    <origin rpy="0 0 0" xyz="0.008005 0.015749 -0.290203"/>
+    <geometry>
+      <mesh filename="package://mvp_arm_6dof_v4_description/meshes/AX12A_servo__2__1.stl" scale="0.001 0.001 0.001"/>
+    </geometry>
+    <material name="silver"/>
+  </visual>
+  <collision>
+    <origin rpy="0 0 0" xyz="0.008005 0.015749 -0.290203"/>
+    <geometry>
+      <mesh filename="package://mvp_arm_6dof_v4_description/meshes/AX12A_servo__2__1.stl" scale="0.001 0.001 0.001"/>
+    </geometry>
+  </collision>
+</link>
+<link name="f2Bracket__1__1">
+  <inertial>
+    <origin rpy="0 0 0" xyz="-2.7952998737051964e-06 0.020999000000009316 0.016208265438762803"/>
+    <mass value="0.0037556666472927302"/>
+    <inertia ixx="2e-06" ixy="-0.0" ixz="0.0" iyy="1e-06" iyz="0.0" izz="1e-06"/>
+  </inertial>
+  <visual>
+    <origin rpy="0 0 0" xyz="5e-06 0.020499 -0.326203"/>
+    <geometry>
+      <mesh filename="package://mvp_arm_6dof_v4_description/meshes/f2Bracket__1__1.stl" scale="0.001 0.001 0.001"/>
+    </geometry>
+    <material name="silver"/>
+  </visual>
+  <collision>
+    <origin rpy="0 0 0" xyz="5e-06 0.020499 -0.326203"/>
+    <geometry>
+      <mesh filename="package://mvp_arm_6dof_v4_description/meshes/f2Bracket__1__1.stl" scale="0.001 0.001 0.001"/>
+    </geometry>
+  </collision>
+</link>
+<link name="axis3-4_connector__1">
+  <inertial>
+    <origin rpy="0 0 0" xyz="-0.007929416125064691 7.741765706693708e-09 0.02400003895587355"/>
+    <mass value="0.2107220147290529"/>
+    <inertia ixx="0.000105" ixy="0.0" ixz="-0.0" iyy="0.000131" iyz="-0.0" izz="8e-05"/>
+  </inertial>
+  <visual>
+    <origin rpy="0 0 0" xyz="9e-06 -0.0005 -0.352657"/>
+    <geometry>
+      <mesh filename="package://mvp_arm_6dof_v4_description/meshes/axis3-4_connector__1.stl" scale="0.001 0.001 0.001"/>
+    </geometry>
+    <material name="silver"/>
+  </visual>
+  <collision>
+    <origin rpy="0 0 0" xyz="9e-06 -0.0005 -0.352657"/>
+    <geometry>
+      <mesh filename="package://mvp_arm_6dof_v4_description/meshes/axis3-4_connector__1.stl" scale="0.001 0.001 0.001"/>
+    </geometry>
+  </collision>
+</link>
+<link name="f3Bracket__4__1">
+  <inertial>
+    <origin rpy="0 0 0" xyz="-0.008000182448553526 5.293942367812221e-15 0.0018414263829612532"/>
+    <mass value="0.0016262220015435807"/>
+    <inertia ixx="0.0" ixy="-0.0" ixz="-0.0" iyy="0.0" iyz="0.0" izz="0.0"/>
+  </inertial>
+  <visual>
+    <origin rpy="0 0 0" xyz="-0.015991 -0.0005 -0.357657"/>
+    <geometry>
+      <mesh filename="package://mvp_arm_6dof_v4_description/meshes/f3Bracket__4__1.stl" scale="0.001 0.001 0.001"/>
+    </geometry>
+    <material name="silver"/>
+  </visual>
+  <collision>
+    <origin rpy="0 0 0" xyz="-0.015991 -0.0005 -0.357657"/>
+    <geometry>
+      <mesh filename="package://mvp_arm_6dof_v4_description/meshes/f3Bracket__4__1.stl" scale="0.001 0.001 0.001"/>
+    </geometry>
+  </collision>
+</link>
+<link name="f3Bracket__5__1">
+  <inertial>
+    <origin rpy="0 0 0" xyz="-0.008000182448552978 2.045510028719777e-14 -0.0018413484712136996"/>
+    <mass value="0.0016262220015435807"/>
+    <inertia ixx="0.0" ixy="-0.0" ixz="0.0" iyy="0.0" iyz="0.0" izz="0.0"/>
+  </inertial>
+  <visual>
+    <origin rpy="0 0 0" xyz="-0.015991 -0.0005 -0.395657"/>
+    <geometry>
+      <mesh filename="package://mvp_arm_6dof_v4_description/meshes/f3Bracket__5__1.stl" scale="0.001 0.001 0.001"/>
+    </geometry>
+    <material name="silver"/>
+  </visual>
+  <collision>
+    <origin rpy="0 0 0" xyz="-0.015991 -0.0005 -0.395657"/>
+    <geometry>
+      <mesh filename="package://mvp_arm_6dof_v4_description/meshes/f3Bracket__5__1.stl" scale="0.001 0.001 0.001"/>
+    </geometry>
+  </collision>
+</link>
+<link name="AX12A_servo__3__1">
+  <inertial>
+    <origin rpy="0 0 0" xyz="-0.014794153871849637 -0.005876867522647733 -0.013500670403273962"/>
+    <mass value="0.3366787209762054"/>
+    <inertia ixx="8.2e-05" ixy="-1e-06" ixz="0.0" iyy="5.4e-05" iyz="0.0" izz="9.7e-05"/>
+  </inertial>
+  <visual>
+    <origin rpy="0 0 0" xyz="-0.02399 -0.0085 -0.390157"/>
+    <geometry>
+      <mesh filename="package://mvp_arm_6dof_v4_description/meshes/AX12A_servo__3__1.stl" scale="0.001 0.001 0.001"/>
+    </geometry>
+    <material name="silver"/>
+  </visual>
+  <collision>
+    <origin rpy="0 0 0" xyz="-0.02399 -0.0085 -0.390157"/>
+    <geometry>
+      <mesh filename="package://mvp_arm_6dof_v4_description/meshes/AX12A_servo__3__1.stl" scale="0.001 0.001 0.001"/>
+    </geometry>
+  </collision>
+</link>
+<link name="f3Bracket__6__1">
+  <inertial>
+    <origin rpy="0 0 0" xyz="0.001841704978532227 1.7305601396344628e-14 3.8955867198708916e-08"/>
+    <mass value="0.0016262220015435807"/>
+    <inertia ixx="0.0" ixy="0.0" ixz="0.0" iyy="0.0" iyz="0.0" izz="0.0"/>
+  </inertial>
+  <visual>
+    <origin rpy="0 0 0" xyz="-0.02874 -0.01525 -0.376657"/>
+    <geometry>
+      <mesh filename="package://mvp_arm_6dof_v4_description/meshes/f3Bracket__6__1.stl" scale="0.001 0.001 0.001"/>
+    </geometry>
+    <material name="silver"/>
+  </visual>
+  <collision>
+    <origin rpy="0 0 0" xyz="-0.02874 -0.01525 -0.376657"/>
+    <geometry>
+      <mesh filename="package://mvp_arm_6dof_v4_description/meshes/f3Bracket__6__1.stl" scale="0.001 0.001 0.001"/>
+    </geometry>
+  </collision>
+</link>
+<link name="axis4ARM__1">
+  <inertial>
+    <origin rpy="0 0 0" xyz="0.0750003175514446 3.053980679457169e-14 3.895587269431289e-08"/>
+    <mass value="0.9125625000000004"/>
+    <inertia ixx="0.000121" ixy="-0.0" ixz="-0.0" iyy="0.001759" iyz="-0.0" izz="0.001784"/>
+  </inertial>
+  <visual>
+    <origin rpy="0 0 0" xyz="-0.030328 -0.01525 -0.376657"/>
+    <geometry>
+      <mesh filename="package://mvp_arm_6dof_v4_description/meshes/axis4ARM__1.stl" scale="0.001 0.001 0.001"/>
+    </geometry>
+    <material name="silver"/>
+  </visual>
+  <collision>
+    <origin rpy="0 0 0" xyz="-0.030328 -0.01525 -0.376657"/>
+    <geometry>
+      <mesh filename="package://mvp_arm_6dof_v4_description/meshes/axis4ARM__1.stl" scale="0.001 0.001 0.001"/>
+    </geometry>
+  </collision>
+</link>
+<link name="f3Bracket__7__1">
+  <inertial>
+    <origin rpy="0 0 0" xyz="0.0018417049785319495 4.3933606752588616e-14 3.895586681013086e-08"/>
+    <mass value="0.0016262220015435807"/>
+    <inertia ixx="0.0" ixy="0.0" ixz="0.0" iyy="0.0" iyz="0.0" izz="0.0"/>
+  </inertial>
+  <visual>
+    <origin rpy="0 0 0" xyz="-0.180328 -0.01525 -0.376657"/>
+    <geometry>
+      <mesh filename="package://mvp_arm_6dof_v4_description/meshes/f3Bracket__7__1.stl" scale="0.001 0.001 0.001"/>
+    </geometry>
+    <material name="silver"/>
+  </visual>
+  <collision>
+    <origin rpy="0 0 0" xyz="-0.180328 -0.01525 -0.376657"/>
+    <geometry>
+      <mesh filename="package://mvp_arm_6dof_v4_description/meshes/f3Bracket__7__1.stl" scale="0.001 0.001 0.001"/>
+    </geometry>
+  </collision>
+</link>
+<link name="AX12A_servo__4__1">
+  <inertial>
+    <origin rpy="0 0 0" xyz="0.023373450028783493 -0.014794971423247538 -0.00799925168497867"/>
+    <mass value="0.3366787209762054"/>
+    <inertia ixx="5.4e-05" ixy="-1e-06" ixz="-0.0" iyy="8.2e-05" iyz="-0.0" izz="9.7e-05"/>
+  </inertial>
+  <visual>
+    <origin rpy="0 0 0" xyz="-0.185828 -0.03125 -0.384657"/>
+    <geometry>
+      <mesh filename="package://mvp_arm_6dof_v4_description/meshes/AX12A_servo__4__1.stl" scale="0.001 0.001 0.001"/>
+    </geometry>
+    <material name="silver"/>
+  </visual>
+  <collision>
+    <origin rpy="0 0 0" xyz="-0.185828 -0.03125 -0.384657"/>
+    <geometry>
+      <mesh filename="package://mvp_arm_6dof_v4_description/meshes/AX12A_servo__4__1.stl" scale="0.001 0.001 0.001"/>
+    </geometry>
+  </collision>
+</link>
+<link name="f2Bracket__2__1">
+  <inertial>
+    <origin rpy="0 0 0" xyz="0.016208313512270894 -0.020999999999945295 -3.165119723091969e-06"/>
+    <mass value="0.0037556666472927302"/>
+    <inertia ixx="1e-06" ixy="0.0" ixz="0.0" iyy="1e-06" iyz="0.0" izz="2e-06"/>
+  </inertial>
+  <visual>
+    <origin rpy="0 0 0" xyz="-0.221828 -0.036 -0.376657"/>
+    <geometry>
+      <mesh filename="package://mvp_arm_6dof_v4_description/meshes/f2Bracket__2__1.stl" scale="0.001 0.001 0.001"/>
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